Commit message: Drivers for the system have been created, though some may not be fully implemented.

File: src/andreas_arm_description/urdf/andreas_arm_description.xacro (robot description, xacro)
@@ -185,5 +185,5 @@
         <xacro:defaultInertial mass="1" />
     </link>
-    <joint name="world" type="fixed">
+    <joint name="world_joint" type="fixed">
         <parent link="world" />
         <child link="base_link" />
