Commit message: Changes to allow for the scorbot-er III to be used with the system

File: src/andreas_arm_description/urdf/sboter4u_model.xacro (robot description, xacro)
@@ -1,4 +1,18 @@
 <?xml version="1.0"?>
 <robot xmlns:xacro="http://www.ros.org/wiki/xacro" name="sboter4u_model">
+  <xacro:macro name="defaultInertial" params="mass">
+    <inertial>
+      <mass value="${mass}" />
+      <inertia
+        ixx="1.0"
+        ixy="0.0"
+        ixz="0.0"
+        iyy="1.0"
+        iyz="0.0"
+        izz="1.0" />
+    </inertial>
+  </xacro:macro>
+  <link
+      name="world" />
   <link
     name="base_Link">
@@ -23,5 +37,5 @@
       <geometry>
         <mesh
-          filename="package://sboter4u_model/meshes/base_Link.STL" />
+          filename="package://andreas_arm_description/meshes/base_Link.STL" />
       </geometry>
       <material
@@ -37,8 +51,13 @@
       <geometry>
         <mesh
-          filename="package://sboter4u_model/meshes/base_Link.STL" />
-      </geometry>
-    </collision>
-  </link>
+          filename="package://andreas_arm_description/meshes/base_Link.STL" />
+      </geometry>
+    </collision>
+    <xacro:defaultInertial mass="1" />
+  </link>
+  <joint name="world_joint" type="fixed">
+    <parent link="world" />
+    <child link="base_Link" />
+  </joint>
   <link
     name="shoulder_Link">
@@ -63,5 +82,5 @@
       <geometry>
         <mesh
-          filename="package://sboter4u_model/meshes/shoulder_Link.STL" />
+          filename="package://andreas_arm_description/meshes/shoulder_Link.STL" />
       </geometry>
       <material
@@ -77,7 +96,8 @@
       <geometry>
         <mesh
-          filename="package://sboter4u_model/meshes/shoulder_Link.STL" />
-      </geometry>
-    </collision>
+          filename="package://andreas_arm_description/meshes/shoulder_Link.STL" />
+      </geometry>
+    </collision>
+    <xacro:defaultInertial mass="1" />
   </link>
   <joint
@@ -102,4 +122,14 @@
       friction="0.01" />
   </joint>
+  <transmission name="baseTransmission">
+    <type>transmission_interface/SimpleTransmission</type>
+    <joint name="base_joint" type="SimpleTransmission">
+      <hardwareInterface>EffortJointInterface</hardwareInterface>
+    </joint>
+    <actuator name="base_motor">
+      <machanicalReduction>1</machanicalReduction>
+      <hardwareInterface>EffortJointInterface</hardwareInterface>
+    </actuator>
+  </transmission>
   <link
     name="elbow_Link">
@@ -124,5 +154,5 @@
       <geometry>
         <mesh
-          filename="package://sboter4u_model/meshes/elbow_Link.STL" />
+          filename="package://andreas_arm_description/meshes/elbow_Link.STL" />
       </geometry>
       <material
@@ -138,7 +168,8 @@
       <geometry>
         <mesh
-          filename="package://sboter4u_model/meshes/elbow_Link.STL" />
-      </geometry>
-    </collision>
+          filename="package://andreas_arm_description/meshes/elbow_Link.STL" />
+      </geometry>
+    </collision>
+    <xacro:defaultInertial mass="1" />
   </link>
   <joint
@@ -163,4 +194,14 @@
       friction="0.01" />
   </joint>
+  <transmission name="shoulderTransmission">
+    <type>transmission_interface/SimpleTransmission</type>
+    <joint name="shoulder_joint" type="SimpleTransmission">
+      <hardwareInterface>EffortJointInterface</hardwareInterface>
+    </joint>
+    <actuator name="shoulder_motor">
+      <machanicalReduction>1</machanicalReduction>
+      <hardwareInterface>EffortJointInterface</hardwareInterface>
+    </actuator>
+  </transmission>
   <link
     name="pitch_Link">
@@ -185,5 +226,5 @@
       <geometry>
         <mesh
-          filename="package://sboter4u_model/meshes/pitch_Link.STL" />
+          filename="package://andreas_arm_description/meshes/pitch_Link.STL" />
       </geometry>
       <material
@@ -199,7 +240,8 @@
       <geometry>
         <mesh
-          filename="package://sboter4u_model/meshes/pitch_Link.STL" />
-      </geometry>
-    </collision>
+          filename="package://andreas_arm_description/meshes/pitch_Link.STL" />
+      </geometry>
+    </collision>
+    <xacro:defaultInertial mass="1" />
   </link>
   <joint
@@ -224,4 +266,14 @@
       friction="0.01" />
   </joint>
+  <transmission name="elbowTransmission">
+    <type>transmission_interface/SimpleTransmission</type>
+    <joint name="elbow_joint" type="SimpleTransmission">
+      <hardwareInterface>EffortJointInterface</hardwareInterface>
+    </joint>
+    <actuator name="elbow_motor">
+      <machanicalReduction>1</machanicalReduction>
+      <hardwareInterface>EffortJointInterface</hardwareInterface>
+    </actuator>
+  </transmission>
   <link
     name="roll_Link">
@@ -246,5 +298,5 @@
       <geometry>
         <mesh
-          filename="package://sboter4u_model/meshes/roll_Link.STL" />
+          filename="package://andreas_arm_description/meshes/roll_Link.STL" />
       </geometry>
       <material
@@ -260,7 +312,8 @@
       <geometry>
         <mesh
-          filename="package://sboter4u_model/meshes/roll_Link.STL" />
-      </geometry>
-    </collision>
+          filename="package://andreas_arm_description/meshes/roll_Link.STL" />
+      </geometry>
+    </collision>
+    <xacro:defaultInertial mass="1" />
   </link>
   <joint
@@ -285,4 +338,14 @@
       friction="0.01" />
   </joint>
+  <transmission name="pitchTransmission">
+    <type>transmission_interface/SimpleTransmission</type>
+    <joint name="pitch_joint" type="SimpleTransmission">
+      <hardwareInterface>EffortJointInterface</hardwareInterface>
+    </joint>
+    <actuator name="pitch_motor">
+      <machanicalReduction>1</machanicalReduction>
+      <hardwareInterface>EffortJointInterface</hardwareInterface>
+    </actuator>
+  </transmission>
   <link
     name="gripper_Link">
@@ -307,5 +370,5 @@
       <geometry>
         <mesh
-          filename="package://sboter4u_model/meshes/gripper_Link.STL" />
+          filename="package://andreas_arm_description/meshes/gripper_Link.STL" />
       </geometry>
       <material
@@ -321,7 +384,8 @@
       <geometry>
         <mesh
-          filename="package://sboter4u_model/meshes/gripper_Link.STL" />
-      </geometry>
-    </collision>
+          filename="package://andreas_arm_description/meshes/gripper_Link.STL" />
+      </geometry>
+    </collision>
+    <xacro:defaultInertial mass="1" />
   </link>
   <joint
@@ -346,4 +410,14 @@
       friction="0.01" />
   </joint>
+  <transmission name="rollTransmission">
+    <type>transmission_interface/SimpleTransmission</type>
+    <joint name="roll_joint" type="SimpleTransmission">
+      <hardwareInterface>EffortJointInterface</hardwareInterface>
+    </joint>
+    <actuator name="roll_motor">
+      <machanicalReduction>1</machanicalReduction>
+      <hardwareInterface>EffortJointInterface</hardwareInterface>
+    </actuator>
+  </transmission>
   <link
     name="pad1_Link">
@@ -368,5 +442,5 @@
       <geometry>
         <mesh
-          filename="package://sboter4u_model/meshes/pad1_Link.STL" />
+          filename="package://andreas_arm_description/meshes/pad1_Link.STL" />
       </geometry>
       <material
@@ -382,7 +456,8 @@
       <geometry>
         <mesh
-          filename="package://sboter4u_model/meshes/pad1_Link.STL" />
-      </geometry>
-    </collision>
+          filename="package://andreas_arm_description/meshes/pad1_Link.STL" />
+      </geometry>
+    </collision>
+    <xacro:defaultInertial mass="1" />
   </link>
   <joint
@@ -407,4 +482,14 @@
       friction="0.01" />
   </joint>
+  <transmission name="pad1Transmission">
+    <type>transmission_interface/SimpleTransmission</type>
+    <joint name="pad1_joint" type="SimpleTransmission">
+      <hardwareInterface>EffortJointInterface</hardwareInterface>
+    </joint>
+    <actuator name="pad1_motor">
+      <machanicalReduction>1</machanicalReduction>
+      <hardwareInterface>EffortJointInterface</hardwareInterface>
+    </actuator>
+  </transmission>
   <link
     name="pad2_Link">
@@ -429,5 +514,5 @@
       <geometry>
         <mesh
-          filename="package://sboter4u_model/meshes/pad2_Link.STL" />
+          filename="package://andreas_arm_description/meshes/pad2_Link.STL" />
       </geometry>
       <material
@@ -443,7 +528,8 @@
       <geometry>
         <mesh
-          filename="package://sboter4u_model/meshes/pad2_Link.STL" />
-      </geometry>
-    </collision>
+          filename="package://andreas_arm_description/meshes/pad2_Link.STL" />
+      </geometry>
+    </collision>
+    <xacro:defaultInertial mass="1" />
   </link>
   <joint
@@ -468,3 +554,19 @@
       friction="0.01" />
   </joint>
+  <transmission name="pad2Transmission">
+    <type>transmission_interface/SimpleTransmission</type>
+    <joint name="pad2_joint" type="SimpleTransmission">
+      <hardwareInterface>EffortJointInterface</hardwareInterface>
+    </joint>
+    <actuator name="pad2_motor">
+      <machanicalReduction>1</machanicalReduction>
+      <hardwareInterface>EffortJointInterface</hardwareInterface>
+    </actuator>
+  </transmission>
+    <!-- Gazebo plugin for ROS Control -->
+    <gazebo>
+        <plugin name="gazebo_ros_control" filename="libgazebo_ros_control.so">
+            <robotNamespace>/sboter4u</robotNamespace>
+        </plugin>
+    </gazebo>
 </robot>
